Commit message: 200323

File: urdf/fingertest.xacro (robot description, xacro)
@@ -3,8 +3,9 @@
      Commit Version: 1.5.1-0-g916b5db  Build Version: 1.5.7152.31018
      For more information, please see http://wiki.ros.org/sw_urdf_exporter -->
-<robot name="fingertest" xmlns:xacro="http://ros.org/wiki/xacro">
-  <include filename="$(find fingertest)/urdf/fingertest.gazebo"/>
-  <link
-    name="base_link">
+  <robot name="fingertest" xmlns:xacro="http://www.ros.org/wiki/xacro">
+  <xacro:include filename="$(find fingertest)/urdf/fingertest.gazebo"/>
+  <xacro:macro name="fingertest" params="parent child side *origin">
+  <link
+    name="${side}_base_link">
     <inertial>
       <origin
@@ -46,5 +47,5 @@
   </link>
   <link
-    name="Link_1">
+    name="${side}_Link_1">
     <inertial>
       <origin
@@ -85,18 +86,16 @@
     </collision>
   </link>
-  <link name="world"/>
-  <joint name="fixed456" type="fixed">
-    <origin
-      xyz="0 0 0"
-      rpy="0 0 0" />
-    <parent
-      link="world" />
-    <child
-      link="base_link" />
+  <!-- <link name="world"/> -->
+  <joint name="${side}_fixed456" type="fixed">
+    <xacro:insert_block name="origin" />
+    <parent
+      link="${parent}" />
+    <child
+      link="${side}_base_link" />
     <axis
       xyz="0 0 0" />
   </joint>
   <joint
-    name="Joint1"
+    name="${side}_Joint1"
     type="continuous">
     <origin
@@ -104,12 +103,12 @@
       rpy="0 -0.5235 0" />
     <parent
-      link="base_link" />
-    <child
-      link="Link_1" />
+      link="${side}_base_link" />
+    <child
+      link="${side}_Link_1" />
     <axis
       xyz="0 -1 0" />
   </joint>
   <link
-    name="Link_2">
+    name="${side}_Link_2">
     <inertial>
       <origin
@@ -151,5 +150,5 @@
   </link>
   <joint
-    name="Joint2"
+    name="${side}_Joint2"
     type="continuous">
     <origin
@@ -157,12 +156,12 @@
       rpy="0 0 0" />
     <parent
-      link="Link_1" />
-    <child
-      link="Link_2" />
+      link="${side}_Link_1" />
+    <child
+      link="${side}_Link_2" />
     <axis
       xyz="0 -1 0" />
   </joint>
   <link
-    name="Link_3">
+    name="${side}_Link_3">
     <inertial>
       <origin
@@ -204,5 +203,5 @@
   </link>
   <joint
-    name="Joint3"
+    name="${side}_Joint3"
     type="continuous">
     <origin
@@ -210,39 +209,41 @@
       rpy="0 0.5235 0" />
     <parent
-      link="Link_2" />
-    <child
-      link="Link_3" />
+      link="${side}_Link_2" />
+    <child
+      link="${side}_Link_3" />
     <axis
       xyz="0 -1 0" />
   </joint>
-  <transmission name="tran1">
+  <transmission name="${side}_tran1">
     <type>transmission_interface/SimpleTransmission</type>
-    <joint name="Joint1">
+    <joint name="${side}_Joint1">
       <hardwareInterface>hardware_interface/EffortJointInterface</hardwareInterface>
     </joint>
-    <actuator name="motor1">
+    <actuator name="${side}_motor1">
       <hardwareInterface>hardware_interface/EffortJointInterface</hardwareInterface>
       <mechanicalReduction>1</mechanicalReduction>
     </actuator>
   </transmission>
-    <transmission name="tran2">
+    <transmission name="${side}_tran2">
     <type>transmission_interface/SimpleTransmission</type>
-    <joint name="Joint2">
+    <joint name="${side}_Joint2">
       <hardwareInterface>hardware_interface/EffortJointInterface</hardwareInterface>
     </joint>
-    <actuator name="motor2">
+    <actuator name="${side}_motor2">
       <hardwareInterface>hardware_interface/EffortJointInterface</hardwareInterface>
       <mechanicalReduction>1</mechanicalReduction>
     </actuator>
   </transmission>
-    <transmission name="tran3">
+    <transmission name="${side}_tran3">
     <type>transmission_interface/SimpleTransmission</type>
-    <joint name="Joint3">
+    <joint name="${side}_Joint3">
       <hardwareInterface>hardware_interface/EffortJointInterface</hardwareInterface>
     </joint>
-    <actuator name="motor3">
+    <actuator name="${side}_motor3">
       <hardwareInterface>hardware_interface/EffortJointInterface</hardwareInterface>
       <mechanicalReduction>1</mechanicalReduction>
     </actuator>
   </transmission>
+  <xacro:fingertest_gazebo side="${side}"/>
+  </xacro:macro>
 </robot>
